File: regen-radio/regen-radio.kicad_sch (KiCad schematic)
At the start: 47 parts, among them P1 POTWS20, Q1 2N2219, Q2 2N2219, T1 Antenna-TICKLE-SS, T2 Transformer_1P_1S, U1 LM386

Commit message: feat(regen-radio): assign most footprints to sch
Parts:
- C10, C12, C13, C16, C18, C2, C4, C5, C6, C9: footprint rbg.lab:C_Disc_D10.0mm_W2.5mm_P5.00mm_P1206 -> Capacitor_THT:C_Disc_D10.0mm_W2.5mm_P5.00mm
- L1: footprint rbg.lab:L_Toroid_Vertical_L13.0mm_W6.5mm_P5.60mm -> Inductor_THT:L_Toroid_Vertical_L13.0mm_W6.5mm_P5.60mm
- R1, R14: footprint (none) -> Capacitor_THT:C_Disc_D10.0mm_W2.5mm_P5.00mm
Changed lines of the file:
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@@
       (effects (font (size 1.27 1.27)))
     )
-    (property "Footprint" "rbg.lab:C_Disc_D10.0mm_W2.5mm_P5.00mm_P1206" (at 184.15 85.09 0)
+    (property "Footprint" "Capacitor_THT:C_Disc_D10.0mm_W2.5mm_P5.00mm" (at 184.15 85.09 0)
       (effects (font (size 1.27 1.27)) hide)
     )
@@
       (effects (font (size 1.27 1.27)))
     )
-    (property "Footprint" "rbg.lab:C_Disc_D10.0mm_W2.5mm_P5.00mm_P1206" (at 97.79 63.5 0)
+    (property "Footprint" "Capacitor_THT:C_Disc_D10.0mm_W2.5mm_P5.00mm" (at 97.79 63.5 0)
       (effects (font (size 1.27 1.27)) hide)
     )
@@
       (effects (font (size 1.27 1.27)) (justify right))
     )
-    (property "Footprint" "rbg.lab:C_Disc_D10.0mm_W2.5mm_P5.00mm_P1206" (at 128.27 96.52 0)
+    (property "Footprint" "Capacitor_THT:C_Disc_D10.0mm_W2.5mm_P5.00mm" (at 128.27 96.52 0)
       (effects (font (size 1.27 1.27)) hide)
     )
@@
       (effects (font (size 1.27 1.27)) (justify right))
     )
-    (property "Footprint" "rbg.lab:C_Disc_D10.0mm_W2.5mm_P5.00mm_P1206" (at 86.36 97.79 0)
+    (property "Footprint" "Capacitor_THT:C_Disc_D10.0mm_W2.5mm_P5.00mm" (at 86.36 97.79 0)
       (effects (font (size 1.27 1.27)) hide)
     )
@@
       (effects (font (size 1.27 1.27)) (justify right))
     )
-    (property "Footprint" "" (at 75.184 74.676 90)
+    (property "Footprint" "Capacitor_THT:C_Disc_D10.0mm_W2.5mm_P5.00mm" (at 75.184 74.676 90)
       (effects (font (size 1.27 1.27)) hide)
     )
@@
       (effects (font (size 1.27 1.27)) (justify left))
     )
-    (property "Footprint" "rbg.lab:L_Toroid_Vertical_L13.0mm_W6.5mm_P5.60mm" (at 76.2 52.07 0)
+    (property "Footprint" "Inductor_THT:L_Toroid_Vertical_L13.0mm_W6.5mm_P5.60mm" (at 76.2 52.07 0)
       (effects (font (size 1.27 1.27)) hide)
     )
@@
       (effects (font (size 1.27 1.27)) (justify right))
     )
-    (property "Footprint" "rbg.lab:C_Disc_D10.0mm_W2.5mm_P5.00mm_P1206" (at 224.79 93.98 0)
+    (property "Footprint" "Capacitor_THT:C_Disc_D10.0mm_W2.5mm_P5.00mm" (at 224.79 93.98 0)
       (effects (font (size 1.27 1.27)) hide)
     )
@@
       (effects (font (size 1.27 1.27)) (justify right))
     )
-    (property "Footprint" "rbg.lab:C_Disc_D10.0mm_W2.5mm_P5.00mm_P1206" (at 154.94 96.52 0)
+    (property "Footprint" "Capacitor_THT:C_Disc_D10.0mm_W2.5mm_P5.00mm" (at 154.94 96.52 0)
       (effects (font (size 1.27 1.27)) hide)
     )
@@
       (effects (font (size 1.27 1.27)))
     )
-    (property "Footprint" "" (at 42.164 42.164 90)
+    (property "Footprint" "Capacitor_THT:C_Disc_D10.0mm_W2.5mm_P5.00mm" (at 42.164 42.164 90)
       (effects (font (size 1.27 1.27)) hide)
     )
@@
       (effects (font (size 1.27 1.27)) (justify right))
     )
-    (property "Footprint" "rbg.lab:C_Disc_D10.0mm_W2.5mm_P5.00mm_P1206" (at 233.68 93.98 0)
+    (property "Footprint" "Capacitor_THT:C_Disc_D10.0mm_W2.5mm_P5.00mm" (at 233.68 93.98 0)
       (effects (font (size 1.27 1.27)) hide)
     )
@@
       (effects (font (size 1.27 1.27)))
     )
-    (property "Footprint" "rbg.lab:C_Disc_D10.0mm_W2.5mm_P5.00mm_P1206" (at 66.04 81.28 0)
+    (property "Footprint" "Capacitor_THT:C_Disc_D10.0mm_W2.5mm_P5.00mm" (at 66.04 81.28 0)
       (effects (font (size 1.27 1.27)) hide)
     )
@@
       (effects (font (size 1.27 1.27)) (justify right))
     )
-    (property "Footprint" "rbg.lab:C_Disc_D10.0mm_W2.5mm_P5.00mm_P1206" (at 195.58 90.17 0)
+    (property "Footprint" "Capacitor_THT:C_Disc_D10.0mm_W2.5mm_P5.00mm" (at 195.58 90.17 0)
       (effects (font (size 1.27 1.27)) hide)
     )
@@
       (effects (font (size 1.27 1.27)) (justify right))
     )
-    (property "Footprint" "rbg.lab:C_Disc_D10.0mm_W2.5mm_P5.00mm_P1206" (at 49.53 46.99 0)
-      (effects (font (size 1.27 1.27)) hide)
-    )
+    (property "Footprint" "Capacitor_THT:C_Disc_D10.0mm_W2.5mm_P5.00mm" (at 49.53 46.99 0)
+      (effects (font (size 1.27 1.27)) hide)
+    )

Commit message: fix: assign missing footprints
Parts:
- C7: footprint rbg.lab:Ceramic-C-Trimmer-PTH-D5-P5 -> radio:Film-C-Trimmer-PTH-D7.5-P5.08-3
- T2: footprint rbg.lab:FT50-43-Bifilar -> radio:FT50-43-Bifilar
Changed lines of the file:
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@@
       (effects (font (size 1.778 1.5113)) (justify left bottom))
     )
-    (property "Footprint" "rbg.lab:Ceramic-C-Trimmer-PTH-D5-P5" (at 97.79 76.2 0)
+    (property "Footprint" "radio:Film-C-Trimmer-PTH-D7.5-P5.08-3" (at 97.79 76.2 0)
       (effects (font (size 1.27 1.27)) hide)
     )
@@
       (effects (font (size 1.27 1.27)))
     )
-    (property "Footprint" "rbg.lab:FT50-43-Bifilar" (at 132.08 71.12 0)
-      (effects (font (size 1.27 1.27)) hide)
-    )
+    (property "Footprint" "radio:FT50-43-Bifilar" (at 132.08 71.12 0)
+      (effects (font (size 1.27 1.27)) hide)
+    )
