File: regen-radio/regen-radio.kicad_pcb (KiCad board)
At the start: 2 copper layers, 47 parts, among them P1 POTWS20, Q1 2N2219, Q2 2N2219, T1 Antenna-TICKLE-SS, T2 Transformer_1P_1S, U1 LM386

Commit message: feat: basic layout
Parts:
- moved H4 148.8 mm to (19.3, 109.0)
- moved H1 132.3 mm to (19.3, 19.0)
- moved H3 85.4 mm to (109.3, 109.0)
- moved C18 55.5 mm to (52.9, 106.9)
- moved R14 45.4 mm to (80.6, 31.5), turned to 180 degrees
- moved H2 43.3 mm to (109.3, 19.0)
- moved LS1 42.0 mm to (108.5, 77.5), turned to 90 degrees
- moved U1 41.4 mm to (70.7, 88.7)
- moved C13 38.9 mm to (57.9, 102.4), turned to 180 degrees
- moved C1 38.9 mm to (80.6, 43.4)
- moved R9 33.2 mm to (73.0, 52.1), turned to -90 degrees
- moved R8 32.8 mm to (65.1, 87.1), turned to -90 degrees
- moved C8 32.3 mm to (80.6, 55.1)
- moved R10 31.5 mm to (52.9, 79.8), turned to -90 degrees
- moved D2 31.3 mm to (66.4, 78.8), turned to 180 degrees
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Routing:
- net Net-(D1-K): track 0.00 -> 89.3 mm
- net VCC: track 0.00 -> 80.9 mm
- net Net-(C19-Pad1): track 0.00 -> 49.9 mm
- net Net-(C14-Pad1): track 0.00 -> 44.5 mm
- net Net-(D2-A): track 0.00 -> 40.1 mm
- net Net-(Q1-B): track 0.00 -> 32.3 mm
- net Net-(Q2-B): track 0.00 -> 28.4 mm
- net Net-(U1--): track 0.00 -> 28.2 mm
- net Net-(U1-BYPASS): track 0.00 -> 27.1 mm
- net Net-(Q1-E): track 0.00 -> 25.7 mm
- net Net-(Q2-C): track 0.00 -> 22.0 mm
- net Net-(Q2-E): track 0.00 -> 17.4 mm
- net Net-(C11-Pad2): track 0.00 -> 14.3 mm
- net Net-(P1-Pad1): track 0.00 -> 13.8 mm
- net Net-(D2-K): track 0.00 -> 12.7 mm
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- added copper zone on B.Cu, net GND
- added copper zone on F.Cu, net GND
Other:
- board outline added: 100 x 100 mm
